Commit message: add support of socket can, but it still not work, seems the write part noe work

File: src/allegro_hand_ros_v4/src/allegro_hand_description/allegro_hand_description_right.urdf (robot description, URDF)
Before this commit: robot allegro_hand_right, 21 links, 20 joints
Links:
- removed link link_0.0
- removed link link_1.0
- removed link link_10.0
- removed link link_11.0
- removed link link_11.0_tip
- removed link link_12.0
- removed link link_13.0
- removed link link_14.0
- removed link link_15.0
- removed link link_15.0_tip
- removed link link_2.0
- removed link link_3.0
- removed link link_3.0_tip
- removed link link_4.0
- removed link link_5.0
- removed link link_6.0
- removed link link_7.0
- removed link link_7.0_tip
- removed link link_8.0
- removed link link_9.0
- added link base_link
- added link link_0, mass 0.0119; collision box size=0.0196 0.0275 0.0164; visual mesh filename=package://allegro_hand_description/meshes/link_0.0.STL
- added link link_1, mass 0.065; collision box size=0.0196 0.0275 0.054; visual mesh filename=package://allegro_hand_description/meshes/link_1.0.STL
- added link link_10, mass 0.0355; collision box size=0.0196 0.0275 0.0384; visual mesh filename=package://allegro_hand_description/meshes/link_2.0.STL
- added link link_11, mass 0.0096; collision box size=0.0196 0.0275 0.026699999999999998; visual mesh filename=package://allegro_hand_description/meshes/link_3.0.STL
- added link link_11_tip, mass 0.0168; collision sphere radius=0.012; visual mesh filename=package://allegro_hand_description/meshes/link_3.0_tip.STL
- added link link_12, mass 0.0176; collision box size=0.0358 0.034 0.0455; visual mesh filename=package://allegro_hand_description/meshes/link_12.0_right.S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
- added link link_13, mass 0.0119; collision box size=0.0196 0.0275 0.0177; visual mesh filename=package://allegro_hand_description/meshes/link_13.0.STL
- added link link_14, mass 0.038; collision box size=0.0196 0.0275 0.0514; visual mesh filename=package://allegro_hand_description/meshes/link_14.0.STL
- added link link_15, mass 0.0388; collision box size=0.0196 0.0275 0.042300000000000004; visual mesh filename=package://allegro_hand_description/meshes/link_15.0.STL
- added link link_15_tip, mass 0.0168; collision sphere radius=0.012; visual mesh filename=package://allegro_hand_description/meshes/link_15.0_tip.STL
- added link link_2, mass 0.0355; collision box size=0.0196 0.0275 0.0384; visual mesh filename=package://allegro_hand_description/meshes/link_2.0.STL
- added link link_3, mass 0.0096; collision box size=0.0196 0.0275 0.026699999999999998; visual mesh filename=package://allegro_hand_description/meshes/link_3.0.STL
- added link link_3_tip, mass 0.0168; collision sphere radius=0.012; visual mesh filename=package://allegro_hand_description/meshes/link_3.0_tip.STL
- added link link_4, mass 0.0119; collision box size=0.0196 0.0275 0.0164; visual mesh filename=package://allegro_hand_description/meshes/link_0.0.STL
- added link link_5, mass 0.065; collision box size=0.0196 0.0275 0.054; visual mesh filename=package://allegro_hand_description/meshes/link_1.0.STL
- added link link_6, mass 0.0355; collision box size=0.0196 0.0275 0.0384; visual mesh filename=package://allegro_hand_description/meshes/link_2.0.STL
- added link link_7, mass 0.0096; collision box size=0.0196 0.0275 0.026699999999999998; visual mesh filename=package://allegro_hand_description/meshes/link_3.0.STL
- added link link_7_tip, mass 0.0168; collision sphere radius=0.012; visual mesh filename=package://allegro_hand_description/meshes/link_3.0_tip.STL
- added link link_8, mass 0.0119; collision box size=0.0196 0.0275 0.0164; visual mesh filename=package://allegro_hand_description/meshes/link_0.0.STL
- added link link_9, mass 0.065; collision box size=0.0196 0.0275 0.054; visual mesh filename=package://allegro_hand_description/meshes/link_1.0.STL
- added link world
Joints:
- removed joint joint_11.0_tip
- removed joint joint_15.0_tip
- removed joint joint_3.0_tip
- removed joint joint_7.0_tip
- added joint base_link_to_palm: type fixed, parent base_link, child palm_link
- added joint joint_11_tip: type fixed, parent link_11, child link_11_tip, origin xyz=0 0 0.026699999999999998 rpy=0 0 0
- added joint joint_15_tip: type fixed, parent link_15, child link_15_tip, origin xyz=0 0 0.042300000000000004 rpy=0 0 0
- added joint joint_3_tip: type fixed, parent link_3, child link_3_tip, origin xyz=0 0 0.026699999999999998 rpy=0 0 0
- added joint joint_7_tip: type fixed, parent link_7, child link_7_tip, origin xyz=0 0 0.026699999999999998 rpy=0 0 0
- added joint world_to_base_link=: type fixed, parent world, child base_link
- joint joint_0.0: child link_0.0 -> link_0; origin xyz=0 0.0435 -0.001542 rpy=-0.08726646255 0 0 -> xyz=0 0.0435 -0.001542 rpy=-0.08726646254999999 0 0
- joint joint_1.0: child link_1.0 -> link_1; limit lower=-0.196 upper=1.61 effort=15 velocity=7 -> lower=-0.19599999999999998 upper=1.6099999999999999 effort=15 velocity=7; parent link_0.0 -> link_0
- joint joint_10.0: child link_10.0 -> link_10; limit lower=-0.174 upper=1.709 effort=15 velocity=7 -> lower=-0.17400000000000002 upper=1.7089999999999999 effort=15 velocity=7; parent link_9.0 -> link_9
- joint joint_11.0: child link_11.0 -> link_11; limit lower=-0.227 upper=1.618 effort=15 velocity=7 -> lower=-0.227 upper=1.6179999999999999 effort=15 velocity=7; parent link_10.0 -> link_10
- joint joint_12.0: child link_12.0 -> link_12; origin xyz=-0.0182 0.019333 -0.045987 rpy=0 -1.65806278845 -1.5707963259 -> xyz=-0.0182 0.019333 -0.045987 rpy=0 -1.6580627884499999 -1.5707963259
- joint joint_13.0: child link_13.0 -> link_13; limit lower=-0.105 upper=1.163 effort=15 velocity=7 -> lower=-0.10499999999999998 upper=1.1629999999999998 effort=15 velocity=7; parent link_12.0 -> link_12
- joint joint_14.0: child link_14.0 -> link_14; limit lower=-0.189 upper=1.644 effort=15 velocity=7 -> lower=-0.18899999999999997 upper=1.644 effort=15 velocity=7; parent link_13.0 -> link_13
- joint joint_15.0: child link_15.0 -> link_15; limit lower=-0.162 upper=1.719 effort=15 velocity=7 -> lower=-0.162 upper=1.7189999999999999 effort=15 velocity=7; parent link_14.0 -> link_14
- joint joint_2.0: child link_2.0 -> link_2; limit lower=-0.174 upper=1.709 effort=15 velocity=7 -> lower=-0.17400000000000002 upper=1.7089999999999999 effort=15 velocity=7; parent link_1.0 -> link_1
- joint joint_3.0: child link_3.0 -> link_3; limit lower=-0.227 upper=1.618 effort=15 velocity=7 -> lower=-0.227 upper=1.6179999999999999 effort=15 velocity=7; parent link_2.0 -> link_2
- joint joint_4.0: child link_4.0 -> link_4
- joint joint_5.0: child link_5.0 -> link_5; limit lower=-0.196 upper=1.61 effort=15 velocity=7 -> lower=-0.19599999999999998 upper=1.6099999999999999 effort=15 velocity=7; parent link_4.0 -> link_4
- joint joint_6.0: child link_6.0 -> link_6; limit lower=-0.174 upper=1.709 effort=15 velocity=7 -> lower=-0.17400000000000002 upper=1.7089999999999999 effort=15 velocity=7; parent link_5.0 -> link_5
- joint joint_7.0: child link_7.0 -> link_7; limit lower=-0.227 upper=1.618 effort=15 velocity=7 -> lower=-0.227 upper=1.6179999999999999 effort=15 velocity=7; parent link_6.0 -> link_6
- joint joint_8.0: child link_8.0 -> link_8; origin xyz=0 -0.0435 -0.001542 rpy=0.08726646255 0 0 -> xyz=0 -0.0435 -0.001542 rpy=0.08726646254999999 0 0
- joint joint_9.0: child link_9.0 -> link_9; limit lower=-0.196 upper=1.61 effort=15 velocity=7 -> lower=-0.19599999999999998 upper=1.6099999999999999 effort=15 velocity=7; parent link_8.0 -> link_8

File: src/allegro_hand_ros_v4/src/allegro_hand_description/allegro_hand_description_right.xacro (robot description, xacro)
@@ -46,4 +46,14 @@
     <!-- ============================================================================= -->
     <!-- PALM -->
+    <link name="world" />
+    <joint name="world_to_base_link=" type="fixed">
+        <parent link="world"/>
+        <child link="base_link"/>
+    </joint>
+    <link name="base_link" />
+    <joint name="base_link_to_palm" type="fixed">
+        <parent link="base_link"/>
+        <child link="palm_link"/>
+    </joint>
     <link name="palm_link">
         <visual>
@@ -99,5 +109,5 @@
             </inertial>
         </link>
-        <joint name="joint_${finger_num*4+0}.0" type="revolute">
+        <joint name="joint_${finger_num*4+0}_revo" type="revolute">
             <axis xyz="-1 0 0"/>
             <limit effort="15" velocity="7"
@@ -134,5 +144,5 @@
             </inertial>
         </link>
-        <joint name="joint_${finger_num*4+1}.0" type="revolute">
+        <joint name="joint_${finger_num*4+1}_revo" type="revolute">
             <axis xyz="0 0 1"/>
             <limit effort="15" velocity="7"
@@ -166,5 +176,5 @@
             </inertial>
         </link>
-        <joint name="joint_${finger_num*4+2}.0" type="revolute">
+        <joint name="joint_${finger_num*4+2}_revo" type="revolute">
             <axis xyz="0 1 0"/>
             <limit effort="15" velocity="7"
@@ -199,5 +209,5 @@
             </inertial>
         </link>
-        <joint name="joint_${finger_num*4+3}.0" type="revolute">
+        <joint name="joint_${finger_num*4+3}_revo" type="revolute">
             <axis xyz="0 1 0"/>
             <limit effort="15" velocity="7"
@@ -265,5 +275,5 @@
             </inertial>
         </link>
-        <joint name="joint_${finger_num*4+0}.0" type="revolute">
+        <joint name="joint_${finger_num*4+0}_revo" type="revolute">
             <axis xyz="0 0 1"/>
             <limit effort="15" velocity="7"
@@ -298,5 +308,5 @@
             </inertial>
         </link>
-        <joint name="joint_${finger_num*4+1}.0" type="revolute">
+        <joint name="joint_${finger_num*4+1}_revo" type="revolute">
             <limit effort="15" velocity="7"
                    lower="${limit_1_low+joint_safety_margin}"
@@ -330,5 +340,5 @@
             </inertial>
         </link>
-        <joint name="joint_${finger_num*4+2}.0" type="revolute">
+        <joint name="joint_${finger_num*4+2}_revo" type="revolute">
             <axis xyz="0 1 0"/>
             <limit effort="15" velocity="7"
@@ -362,5 +372,5 @@
             </inertial>
         </link>
-        <joint name="joint_${finger_num*4+3}.0" type="revolute">
+        <joint name="joint_${finger_num*4+3}_revo" type="revolute">
             <axis xyz="0 1 0"/>
             <limit effort="15" velocity="7"
